File: pcb/presence_sensor.kicad_sch (KiCad schematic)
At the start: 53 parts, among them J1 SEN0395, J2 USB4105, J3 SM04B-SRSS-TB(LF)(SN), J4 USB4105, Q1 MBT3904DW1, SW1 SW_Push, SW2 SW_Push, U1 ESP32-S2-MINI-1, U2 USBLC6-2P6, U3 AMS1117-3.3, U4 CP2102N-Axx-xQFN24, U5 USBLC6-2P6

Commit message: Removed USB TTL
Parts:
- removed C15: 1u, Capacitor_SMD:C_0603_1608Metric, symbol Device:C_Small
- removed C16: 10u, Capacitor_SMD:C_0805_2012Metric, symbol Device:C_Small
- removed D4: 1N5819, Diode_THT:D_DO-41_SOD81_P10.16mm_Horizontal, symbol Diode:1N5819
- removed FL1, FL2: DLP11SN900HL2L, Presence Sensor:FIL_DLP11SN900HL2L, symbol Presence Sensor:DLP11SN900HL2L
- removed J4: USB4105, Presence Sensor:GCT_USB4105_REVA, symbol Presence Sensor:USB4105
- removed R13, R7: 10K, Resistor_SMD:R_0603_1608Metric, symbol Device:R_Small
- removed R14, R15: 0R, Resistor_SMD:R_0603_1608Metric, symbol Device:R_Small
- removed R18, R19: 5.1K, Resistor_SMD:R_0603_1608Metric, symbol Device:R_Small
- removed R3: 22.1K, Resistor_SMD:R_0603_1608Metric, symbol Device:R_Small
- removed R4: 47.5K, Resistor_SMD:R_0603_1608Metric, symbol Device:R_Small
- removed U2, U5: USBLC6-2P6, Package_TO_SOT_SMD:SOT-666, symbol Power_Protection:USBLC6-2P6
- removed U4: CP2102N-Axx-xQFN24, Package_DFN_QFN:QFN-24-1EP_4x4mm_P0.5mm_EP2.6x2.6mm, symbol Interface_USB:CP2102N-Axx-xQFN24
- added D4: B220, Diode_SMD:D_SMB, symbol Diode:B220
- added D5: ESDA6V1-5SC6, Package_TO_SOT_SMD:SOT-23-6, symbol Power_Protection:ESDA6V1-5SC6
- added FL?: DLP11SN900HL2L, Presence Sensor:FIL_DLP11SN900HL2L, symbol Presence Sensor:DLP11SN900HL2L
- added J4: Conn_01x05, symbol Connector_Generic:Conn_01x05
- added U?: USBLC6-2P6, Package_TO_SOT_SMD:SOT-666, symbol Power_Protection:USBLC6-2P6
Connections:
- net USB_DEV_N is gone; now on net USB_HOST_N: U1.23 (IO19)
- net USB_DEV_P is gone; now on net USB_HOST_P: U1.24 (IO20)
- net +5V: now also D4.1 (K), U?.5 (VBUS)
- net DTR: now also D5.3 (IO2), J4.4 (Pin_4)
- net ESP_RXD: now also D5.4 (IO3), J4.3 (Pin_3)
- net ESP_TXD: now also D5.5 (IO4), J4.2 (Pin_2)
- net GND: now also D5.2 (GND), J4.1 (Pin_1), U?.2 (GND)
- net RTS: now also D5.1 (IO1), J4.5 (Pin_5)
- net USB_CON_N: now also FL?.3, U?.3 (I/O2), U?.4 (I/O2)
- net USB_CON_P: now also FL?.2, U?.1 (I/O1), U?.6 (I/O1)
- net USB_HOST_N: now also FL?.4
- net USB_HOST_P: now also FL?.1
- net VBUS: now also D4.2 (A)
- no-connect marks 15 -> 7

Commit message: Update
Parts:
- removed D4: B220, Diode_SMD:D_SMB, symbol Diode:B220
- added C15, C16, C19, C21, C24: 100n, Capacitor_SMD:C_0603_1608Metric, symbol Device:C_Small
- added C17, C18: 12pF, Capacitor_SMD:C_0603_1608Metric, symbol Device:C_Small
- added C20: 4.7u, Capacitor_SMD:C_0805_2012Metric, symbol Device:C_Small
- added C22: 10u, Capacitor_SMD:C_0805_2012Metric, symbol Device:C_Small
- added C23: 1u, Capacitor_SMD:C_0603_1608Metric, symbol Device:C_Small
- added FID1, FID2, FID3, FID4, FID5, FID6: Fiducial, Fiducial:Fiducial_0.5mm_Mask1mm, symbol Mechanical:Fiducial
- added H1, H2: MountingHole, MountingHole:MountingHole_2.7mm_M2.5, symbol Mechanical:MountingHole
- added H3, H4: MountingHole, MountingHole:MountingHole_2.2mm_M2, symbol Mechanical:MountingHole
- added R13: DNP, Resistor_SMD:R_0603_1608Metric, symbol Device:R_Small
- added R14, R19, R20, R3: 10K, Resistor_SMD:R_0603_1608Metric, symbol Device:R_Small
- added R15: 22.1K, Resistor_SMD:R_0603_1608Metric, symbol Device:R_Small
- added R18: 47.5K, Resistor_SMD:R_0603_1608Metric, symbol Device:R_Small
- added R21, R22: 0R, Resistor_SMD:R_0603_1608Metric, symbol Device:R_Small
- added R4, R7: 4.7K, Resistor_SMD:R_0603_1608Metric, symbol Device:R_Small
- added SW3: SW_SPDT, Button_Switch_SMD:SW_Push_1P1T-SH_NO_CK_KMR2xxG, symbol Switch:SW_SPDT
- added U4: AP2161W, Package_TO_SOT_SMD:SOT-23-5, symbol Power_Management:AP2161W
- added U5: BMP280, Package_LGA:Bosch_LGA-8_2x2.5mm_P0.65mm_ClockwisePinNumbering, symbol Sensor_Pressure:BMP280
- added U6: FSUSB42UMX, Presence Sensor:IC_FSUSB42UMX, symbol Presence Sensor:FSUSB42UMX
- added U7: CP2102N-Axx-xQFN24, Package_DFN_QFN:QFN-24-1EP_4x4mm_P0.5mm_EP2.6x2.6mm, symbol Interface_USB:CP2102N-Axx-xQFN24
- added Y1: 32.768MHz, Presence Sensor:NX3215SA, symbol Device:Crystal
- C3: footprint Capacitor_SMD:C_1206_3216Metric -> Capacitor_SMD:C_0805_2012Metric
- C8: value 100n -> 1u
- J4: footprint (none) -> Connector_PinHeader_2.54mm:PinHeader_1x05_P2.54mm_Vertical
- gave numbers to parts that had none: 2
Connections:
- net +3V3: now also C8.1, C15.1, C16.1, C19.1, C22.1, C24.1, R14.1, R19.1, R4.1, R7.1, U5.2 (CSB), U5.6 (VDDIO), U5.8 (VDD), U6.9 (VCC), U7.5 (VIO), U7.6 (VDD), U7.7 (VREGIN)
- net +5V: now also U4.1 (OUT)
- net DTR: now also U7.23 (~{DTR})
- net EN: no longer C8.1, R8.2
- net ESP_RXD: now also D5.5 (IO4), J4.2 (Pin_2), R21.2; no longer D5.4 (IO3), J4.3 (Pin_3)
- net ESP_TXD: now also D5.4 (IO3), J4.3 (Pin_3), R22.2; no longer D5.5 (IO4), J4.2 (Pin_2)
- net GND: now also C15.2, C16.2, C17.2, C18.2, C19.2, C20.2, C21.2, C22.2, C23.2, C24.2, R13.2, R18.2, R20.2, U4.2 (GND), U5.1 (GND), U5.7 (GND), U6.3 (GND), U6.8 (~{OE}), U7.2 (GND), U7.25 (GND)
- net I2C_SCL: now also R7.2, U5.4 (SCK)
- net I2C_SDA: now also R4.2, U5.3 (SDI)
- net RTS: now also U7.19 (~{RTS})
- net USB_CON_N: now also FL1.4; no longer FL1.3
- net USB_CON_P: now also FL1.1; no longer FL1.2
- net USB_HOST_N: now also FL1.3, U6.2 (D-); no longer FL1.4, U1.23 (IO19)
- net USB_HOST_P: now also FL1.2, U6.1 (D+); no longer FL1.1, U1.24 (IO20)
- net VBUS: now also C20.1, R15.1, R3.1, U4.5 (IN)
- net OSC_SLOW_P: now reaches U1.19 (IO15)
- net OSC_SLOW_P: now also C17.1, Y1.1
- net OSC_SLOW_N: now reaches U1.20 (IO16)
- net OSC_SLOW_N: now also C18.1, Y1.2
- new net: C23.1, R15.2, R18.1, U7.8 (VBUS)
- new net: R13.1, R8.2, U5.5 (SDO)
- new net: R21.1, U7.21 (TXD)
- new net: R20.1, U7.15 (~{SUSPEND})
- new net: R22.1, U7.20 (RXD)
- new net: R19.2, U7.9 (~{RST})
- new net: R3.2, U4.4 (~{EN})
- new net USB_ESP_N: U1.23 (IO19), U6.6 (HSD2-)
- new net USB_ESP_P: U1.24 (IO20), U6.7 (HSD2+)
- new net USB_SELECT: C21.1, R14.2, U6.10 (SEL)
- new net USB_SERIAL_N: U6.4 (HSD1-), U7.4 (D-)
- new net USB_SERIAL_P: U6.5 (HSD1+), U7.3 (D+)
- no-connect marks 7 -> 17
Other:
- note added: "ADDR Sets the I2C address of the BMP280. Open (default) 0x77 Closed 0x76"
- note added: "Bosch BMP280 - Temperature/Humidity/Pressure"
- moved on the sheet: C3, C4, C5, C6, C7, D1, FL1, J2, R5, R6, U2, U3
